File: eagle/ledshields_v2/leds_9dof.brd (EAGLE design)
At the start: 20 x 42 mm, 14 parts, among them U3 PCA9685

Commit message: modified 2nd version pcb designs for milling
Other:
- outline, holes or cut-outs redrawn
Changed lines of the file:
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@@
 <board>
 <plain>
-<wire x1="0" y1="0" x2="20" y2="0" width="0" layer="20"/>
+<wire x1="0" y1="8.2" x2="8.2" y2="0" width="0" layer="20" curve="90"/>
+<wire x1="8.2" y1="0" x2="20" y2="0" width="0" layer="20"/>
 <wire x1="20" y1="0" x2="20" y2="42" width="0" layer="20"/>
-<wire x1="20" y1="42" x2="0" y2="42" width="0" layer="20"/>
-<wire x1="0" y1="42" x2="0" y2="0" width="0" layer="20"/>
+<wire x1="20" y1="42" x2="7.9" y2="42" width="0" layer="20"/>
+<wire x1="7.9" y1="42" x2="0" y2="34.1" width="0" layer="20" curve="90"/>
+<wire x1="0" y1="34.1" x2="0" y2="8.2" width="0" layer="20"/>
 </plain>
 <attributes>
@@
 <wire x1="8" y1="8.6" x2="10.2" y2="8.6" width="0.3" layer="1"/>
 <wire x1="11.5" y1="0.7" x2="7" y2="0.7" width="0.3" layer="1"/>
-<wire x1="7" y1="0.7" x2="0.7" y2="7.1" width="0.3" layer="1"/>
-<wire x1="0.7" y1="7.1" x2="0.7" y2="19.9" width="0.3" layer="1"/>
+<wire x1="0.7" y1="9.9" x2="0.7" y2="19.9" width="0.3" layer="1"/>
 <wire x1="0.7" y1="19.9" x2="1.8" y2="21" width="0.3" layer="1"/>
 <wire x1="1.8" y1="21" x2="2.24" y2="21" width="0.3" layer="1"/>
 <wire x1="2.24" y1="21" x2="1.7" y2="21" width="0.3" layer="1"/>
 <wire x1="1.7" y1="21" x2="0.7" y2="22" width="0.3" layer="1"/>
-<wire x1="0.7" y1="22" x2="0.7" y2="35.8" width="0.3" layer="1"/>
-<wire x1="0.7" y1="35.8" x2="6.2" y2="41.3" width="0.3" layer="1"/>
-<wire x1="6.2" y1="41.3" x2="11.4" y2="41.3" width="0.3" layer="1"/>
+<wire x1="0.7" y1="22" x2="0.7" y2="35" width="0.3" layer="1"/>
+<wire x1="0.7" y1="35" x2="7" y2="41.3" width="0.3" layer="1"/>
+<wire x1="7" y1="41.3" x2="11.4" y2="41.3" width="0.3" layer="1"/>
 <wire x1="11.97" y1="6.83" x2="11.97" y2="5.750675" width="0.3" layer="1"/>
 <wire x1="10.2" y1="8.6" x2="11.97" y2="6.83" width="0.3" layer="1"/>
@@
 <wire x1="11.9" y1="40.320675" x2="11.9" y2="40.8" width="0.3" layer="1"/>
 <wire x1="11.9" y1="40.8" x2="11.4" y2="41.3" width="0.3" layer="1"/>
+<wire x1="7" y1="0.7" x2="6.3" y2="1.4" width="0.3" layer="1"/>
+<wire x1="6.3" y1="1.4" x2="6.3" y2="4.3" width="0.3" layer="1"/>
+<wire x1="6.3" y1="4.3" x2="0.7" y2="9.9" width="0.3" layer="1"/>
 </signal>
 <signal name="PWM0">
