File: eagle/ledshields_v2/leds.brd (EAGLE design)
At the start: 20 x 42 mm, 14 parts, among them J1 J5MM, U3 PCA9685

Commit message: started second custom PCB arduino code
Parts:
- removed J1: J5MM, jumper:05
- added R9: 0, 01_SparkFun:R2512
Connections:
- new net VCC: JP1.2, LED2.BA, LED2.GA, LED2.RA, R9.2, U3.28
- net 3.3V: now also R9.1; no longer J1.1, J1.2, JP1.2, LED2.BA, LED2.GA, LED2.RA, U3.28
Routing:
- net VCC: track 0.00 -> 17.9 mm
- net 3.3V: track 69.3 -> 53.7 mm
- net SCL: track 33.1 -> 37.1 mm
- net GND: track 71.1 -> 74.1 mm
Changed lines of the file:
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@@
 <layers>
 <layer number="1" name="Top" color="4" fill="1" visible="yes" active="yes"/>
-<layer number="16" name="Bottom" color="1" fill="1" visible="no" active="yes"/>
-<layer number="17" name="Pads" color="2" fill="1" visible="no" active="yes"/>
-<layer number="18" name="Vias" color="2" fill="1" visible="no" active="yes"/>
-<layer number="19" name="Unrouted" color="6" fill="1" visible="no" active="yes"/>
-<layer number="20" name="Dimension" color="15" fill="1" visible="no" active="yes"/>
-<layer number="21" name="tPlace" color="7" fill="1" visible="no" active="yes"/>
-<layer number="22" name="bPlace" color="7" fill="1" visible="no" active="yes"/>
-<layer number="23" name="tOrigins" color="15" fill="1" visible="no" active="yes"/>
-<layer number="24" name="bOrigins" color="15" fill="1" visible="no" active="yes"/>
-<layer number="25" name="tNames" color="7" fill="1" visible="no" active="yes"/>
-<layer number="26" name="bNames" color="7" fill="1" visible="no" active="yes"/>
-<layer number="27" name="tValues" color="7" fill="1" visible="no" active="yes"/>
-<layer number="28" name="bValues" color="7" fill="1" visible="no" active="yes"/>
+<layer number="16" name="Bottom" color="1" fill="1" visible="yes" active="yes"/>
+<layer number="17" name="Pads" color="2" fill="1" visible="yes" active="yes"/>
+<layer number="18" name="Vias" color="2" fill="1" visible="yes" active="yes"/>
+<layer number="19" name="Unrouted" color="6" fill="1" visible="yes" active="yes"/>
+<layer number="20" name="Dimension" color="15" fill="1" visible="yes" active="yes"/>
+<layer number="21" name="tPlace" color="7" fill="1" visible="yes" active="yes"/>
+<layer number="22" name="bPlace" color="7" fill="1" visible="yes" active="yes"/>
+<layer number="23" name="tOrigins" color="15" fill="1" visible="yes" active="yes"/>
+<layer number="24" name="bOrigins" color="15" fill="1" visible="yes" active="yes"/>
+<layer number="25" name="tNames" color="7" fill="1" visible="yes" active="yes"/>
+<layer number="26" name="bNames" color="7" fill="1" visible="yes" active="yes"/>
+<layer number="27" name="tValues" color="7" fill="1" visible="yes" active="yes"/>
+<layer number="28" name="bValues" color="7" fill="1" visible="yes" active="yes"/>
 <layer number="29" name="tStop" color="7" fill="3" visible="no" active="yes"/>
 <layer number="30" name="bStop" color="7" fill="6" visible="no" active="yes"/>
@@
 <element name="JP1" library="SparkFun-Connectors" package="1X05" value="" x="5" y="16" rot="R90"/>
 <element name="LED3" library="Mlab_ProEx2015" package="LED_RGB_6PINS" value="LED_RGB_6PINS" x="10.1" y="4" rot="R270"/>
-<element name="J1" library="jumper" package="05" value="J5MM" x="4.9" y="9.7" rot="R270"/>
+<element name="R9" library="01_SparkFun" package="R2512" value="0" x="4.4" y="8.8" rot="R90"/>
 </elements>
 <signals>
@@
 <contactref element="R5" pad="1"/>
 <contactref element="JP1" pad="5"/>
-<wire x1="8.2" y1="9.5" x2="8.4" y2="9.3" width="0.4064" layer="1"/>
 <wire x1="4.97" y1="37.245" x2="5" y2="37.215" width="0.4064" layer="1"/>
 <wire x1="8.4" y1="9.3" x2="8.4" y2="8.1" width="0.3" layer="1"/>
@@
 <wire x1="8.4" y1="13.9" x2="8.4" y2="11.6" width="0.3" layer="1"/>
 <wire x1="8.4" y1="11.6" x2="8.4" y2="9.3" width="0.3" layer="1"/>
-<wire x1="8.2" y1="9.5" x2="4.4" y2="9.5" width="0.3" layer="1"/>
-<wire x1="4.4" y1="9.5" x2="1.4" y2="12.5" width="0.3" layer="1"/>
-<wire x1="1.4" y1="12.5" x2="1.4" y2="22.56" width="0.3" layer="1"/>
+<wire x1="7.3" y1="8.2" x2="2.2" y2="8.2" width="0.3" layer="1"/>
+<wire x1="1.4" y1="8.9" x2="1.4" y2="22.56" width="0.3" layer="1"/>
 <wire x1="1.4" y1="22.56" x2="5" y2="26.16" width="0.3" layer="1"/>
 <wire x1="8.1372" y1="27.125" x2="5.965" y2="27.125" width="0.3" layer="1"/>
@@
 <vertex x="-0.7" y="42.7"/>
 </polygon>
+<wire x1="1.4" y1="8.9" x2="2.2" y2="8.2" width="0.3" layer="1"/>
+<wire x1="7.3" y1="8.2" x2="8.4" y2="9.3" width="0.3" layer="1"/>
 </signal>
 <signal name="A0">
@@
 <contactref element="LED1" pad="RA"/>
 <contactref element="LED1" pad="BA"/>
-<contactref element="U3" pad="28"/>
 <contactref element="C1" pad="A"/>
 <contactref element="LED3" pad="BA"/>
 <contactref element="LED3" pad="GA"/>
 <contactref element="LED3" pad="RA"/>
-<contactref element="LED2" pad="RA"/>
-<contactref element="LED2" pad="GA"/>
-<contactref element="LED2" pad="BA"/>
-<contactref element="J1" pad="2"/>
-<wire x1="8.03" y1="20.999325" x2="8.099325" y2="20.999325" width="0.4064" layer="1"/>
-<wire x1="8.099325" y1="20.999325" x2="8.1" y2="21" width="0.4064" layer="1"/>
-<wire x1="8.1" y1="19.319325" x2="8.03" y2="19.249325" width="0.4064" layer="1"/>
-<contactref element="JP1" pad="2"/>
-<contactref element="J1" pad="1"/>
-<wire x1="4.9" y1="7.16" x2="4.94" y2="7.16" width="0.4064" layer="1"/>
 <wire x1="7.979325" y1="5.8" x2="8.03" y2="5.749325" width="0.4064" layer="1"/>
 <wire x1="4.995" y1="40.07" x2="4.97" y2="40.045" width="0.4064" layer="1"/>
-<wire x1="8.03" y1="19.249325" x2="5.709325" y2="19.249325" width="0.3" layer="1"/>
-<wire x1="5.709325" y1="19.249325" x2="5" y2="18.54" width="0.3" layer="1"/>
-<wire x1="8.1372" y1="25.175" x2="8.03" y2="25.0678" width="0.3" layer="1"/>
-<wire x1="8.03" y1="25.0678" x2="8.03" y2="22.749325" width="0.3" layer="1"/>
-<wire x1="8.03" y1="22.749325" x2="8.03" y2="20.999325" width="0.3" layer="1"/>
-<wire x1="8.03" y1="20.999325" x2="8.03" y2="19.249325" width="0.3" layer="1"/>
-<wire x1="5" y1="18.54" x2="2.8" y2="16.34" width="0.3" layer="1"/>
-<wire x1="2.8" y1="16.34" x2="2.8" y2="14.2" width="0.3" layer="1"/>
-<wire x1="2.8" y1="14.2" x2="4.76" y2="12.24" width="0.3" layer="1"/>
-<wire x1="4.76" y1="12.24" x2="4.9" y2="12.24" width="0.3" layer="1"/>
 <wire x1="8.03" y1="2.249325" x2="8.03" y2="3.999325" width="0.3" layer="1"/>
 <wire x1="8.03" y1="3.999325" x2="8.03" y2="5.749325" width="0.3" layer="1"/>
-<wire x1="7.979325" y1="5.8" x2="6.26" y2="5.8" width="0.3" layer="1"/>
-<wire x1="6.26" y1="5.8" x2="4.9" y2="7.16" width="0.3" layer="1"/>
-<wire x1="4.9" y1="7.16" x2="0.7" y2="11.36" width="0.3" layer="1"/>
-<wire x1="0.7" y1="11.36" x2="0.7" y2="37.7" width="0.3" layer="1"/>
+<wire x1="7.979325" y1="5.8" x2="6.9" y2="5.8" width="0.3" layer="1"/>
+<wire x1="0.7" y1="8" x2="0.7" y2="37.7" width="0.3" layer="1"/>
 <wire x1="0.7" y1="37.7" x2="3.1" y2="40.1" width="0.3" layer="1"/>
 <wire x1="3.1" y1="40.1" x2="4.915" y2="40.1" width="0.3" layer="1"/>
@@
 <wire x1="8.349325" y1="40.07" x2="10.099325" y2="40.07" width="0.3" layer="1"/>
 <wire x1="10.099325" y1="40.07" x2="11.849325" y2="40.07" width="0.3" layer="1"/>
-<wire x1="0.7" y1="11.36" x2="2.8" y2="14.2" width="0" layer="19" extent="1-1"/>
+<wire x1="4.4" y1="6" x2="6.7" y2="6" width="0.3" layer="1"/>
+<wire x1="6.7" y1="6" x2="6.9" y2="5.8" width="0.3" layer="1"/>
+<wire x1="4.4" y1="6" x2="2.6" y2="6" width="0.3" layer="1"/>
+<wire x1="2.6" y1="6" x2="0.7" y2="8" width="0.3" layer="1"/>
+<contactref element="R9" pad="1"/>
 </signal>
 <signal name="PWM0">
@@
 <wire x1="8.5" y1="17.9" x2="7.4" y2="17.9" width="0.3" layer="1"/>
 <wire x1="7.4" y1="17.9" x2="6.8" y2="17.3" width="0.3" layer="1"/>
-<wire x1="6.8" y1="17.3" x2="6.8" y2="11.8" width="0.3" layer="1"/>
-<wire x1="6.8" y1="11.8" x2="5.6" y2="10.6" width="0.3" layer="1"/>
-<wire x1="5.6" y1="10.6" x2="4.2" y2="10.6" width="0.3" layer="1"/>
-<wire x1="4.2" y1="10.6" x2="2.1" y2="12.7" width="0.3" layer="1"/>
-<wire x1="2.1" y1="12.7" x2="2.1" y2="18.18" width="0.3" layer="1"/>
+<wire x1="6.8" y1="17.3" x2="6.8" y2="9.8" width="0.3" layer="1"/>
+<wire x1="6.8" y1="9.8" x2="6.3" y2="9.3" width="0.3" layer="1"/>
+<wire x1="6.3" y1="9.3" x2="2.5" y2="9.3" width="0.3" layer="1"/>
+<wire x1="2.5" y1="9.3" x2="2.1" y2="9.7" width="0.3" layer="1"/>
+<wire x1="2.1" y1="9.7" x2="2.1" y2="18.18" width="0.3" layer="1"/>
 <wire x1="2.1" y1="18.18" x2="5" y2="21.08" width="0.3" layer="1"/>
 </signal>
@@
 <signal name="N$4">
 </signal>
+<signal name="VCC">
+<contactref element="R9" pad="2"/>
+<contactref element="LED2" pad="GA"/>
+<contactref element="LED2" pad="BA"/>
+<contactref element="LED2" pad="RA"/>
+<contactref element="JP1" pad="2"/>
+<contactref element="U3" pad="28"/>
+<wire x1="8.1372" y1="25.175" x2="8.1372" y2="22.856525" width="0.3" layer="1"/>
+<wire x1="8.1372" y1="22.856525" x2="8.03" y2="22.749325" width="0.3" layer="1"/>
+<wire x1="8.03" y1="22.749325" x2="8.03" y2="20.999325" width="0.3" layer="1"/>
+<wire x1="8.03" y1="20.999325" x2="8.03" y2="19.249325" width="0.3" layer="1"/>
+<wire x1="8.03" y1="19.249325" x2="5.709325" y2="19.249325" width="0.3" layer="1"/>
+<wire x1="5.709325" y1="19.249325" x2="5" y2="18.54" width="0.3" layer="1"/>
+<wire x1="5" y1="18.54" x2="4.54" y2="18.54" width="0.3" layer="1"/>
+<wire x1="4.54" y1="18.54" x2="3" y2="17" width="0.3" layer="1"/>
+<wire x1="3" y1="17" x2="3" y2="14.7" width="0.3" layer="1"/>
+<wire x1="3" y1="14.7" x2="4.4" y2="13.3" width="0.3" layer="1"/>
+<wire x1="4.4" y1="13.3" x2="4.4" y2="11.6" width="0.3" layer="1"/>
+</signal>
 </signals>
