File: eagle/ledshields_v2/leds.sch (EAGLE design)
At the start: 14 parts, among them J1 J5MM, U3 PCA9685

Commit message: started second custom PCB arduino code
Parts:
- removed J1: J5MM, jumper:J5MM
- added R9: 0, 01_SparkFun:RESISTOR2512
Connections:
- new net VCC: JP1.2, LED2.BA, LED2.GA, LED2.RA, R9.2, U3.VDD
- net 3.3V: now also R9.1; no longer J1.1, J1.2, JP1.2, LED2.BA, LED2.GA, LED2.RA, U3.VDD
