File: eagle/custom_pcb/IoT_modules_atmega328_kinemata_v1.brd (EAGLE design)
At the start: 60 x 35 mm, 59 parts, among them IC2 4093DT, Q3 MOSFET-P, T1 2N2222, U1 SFW6R-3STE1LF, U2 ATMEGA328P, U3 FT232RL-BASICSSOP, U4 MCP73831, Y2 8MHz

Commit message: some more initial work on the custom PCB
Parts:
- removed INT_DRDYG_GYRO, INT_INT1X_ACCEL, INT_INT2X_MAG: HEADER_1PIN_MALE, MlabPaja_v3:SPRING_LOADED_HEADER_ANGLE_829-22-020-20-002101_DIGIKEY_ED1320-ND
- removed U$2: LIPO_BATTERY400MAH, MlabPaja_v3:LIPO_BATTERY_400MAH
- moved C7 73.7 mm to (5.91, 15.8), flipped to the bottom
- moved C13 72.4 mm to (22.2, 0.18), turned to 180 degrees
- moved R10 68.6 mm to (6.04, 13.2), flipped to the bottom, turned to 180 degrees
- moved U$5 68.1 mm to (17.8, 32.7), flipped to the bottom
- moved D1 66.1 mm to (46.8, 1.71), turned to 180 degrees
- moved Y2 63.7 mm to (29.4, 10.4), turned to 270 degrees
- moved D4 62.9 mm to (46.7, 3.91), turned to 180 degrees
- moved D5 62.0 mm to (46.5, 6.29), turned to 0 degrees
- moved C10 61.7 mm to (14.5, 31.6), turned to 90 degrees
- moved R8 61.2 mm to (45.5, 5.88), flipped to the bottom, turned to 180 degrees
- moved R20 60.8 mm to (9.83, 32.3), turned to 180 degrees
- moved R3 60.3 mm to (46.5, 3.58), flipped to the bottom
- moved R13 59.6 mm to (45.4, 8.56), flipped to the bottom, turned to 180 degrees
- moved R9 58.7 mm to (6.31, 21.7), flipped to the bottom, turned to 180 degrees
- moved R11 58.1 mm to (5.89, 18.5), flipped to the bottom, turned to 180 degrees
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Connections:
- removed net INT0: INT_INT1X_ACCEL.P$1, U2.17
- removed net INT1: INT_DRDYG_GYRO.P$1, U2.2
- net INT2: no longer INT_INT2X_MAG.P$1
Routing:
- net GND: track 0.00 -> 126.6 mm, vias 0 -> 2
- net 3.3V: track 0.00 -> 87.7 mm, vias 0 -> 3
- net N$13: track 0.00 -> 59.6 mm, vias 0 -> 1
- net 5V: track 0.00 -> 53.8 mm, vias 0 -> 3
- net SCL: track 0.00 -> 50.2 mm
- net SDA: track 0.00 -> 40.7 mm, vias 0 -> 4
- net IS_CON: track 0.00 -> 34.5 mm, vias 0 -> 3
- net KILL: track 0.00 -> 30.6 mm, vias 0 -> 2
- net VIBE: track 0.00 -> 30.1 mm, vias 0 -> 3
- net TX: track 0.00 -> 28.6 mm, vias 0 -> 2
- net BT_RX: track 0.00 -> 26.7 mm, vias 0 -> 2
- net D-USB: track 0.00 -> 21.1 mm, vias 0 -> 1
- net D+USB: track 0.00 -> 19.4 mm, vias 0 -> 1
- net N$19: track 0.00 -> 12.3 mm
- net RXLED: track 0.00 -> 12.2 mm, vias 0 -> 1
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Other:
- board size 60 x 35 mm -> 50 x 35 mm
