File: eagle/custom_pcb/IoT_modules_atmega328_kinemata_v1.sch (EAGLE design)
At the start: 59 parts, among them IC2 4093DT, Q3 MOSFET-P, T1 2N2222, U1 SFW6R-3STE1LF, U2 ATMEGA328P, U3 FT232RL-BASICSSOP, U4 MCP73831, Y2 8MHz

Commit message: some more initial work on the custom PCB
Parts:
- removed INT_DRDYG_GYRO, INT_INT1X_ACCEL, INT_INT2X_MAG: HEADER_1PIN_MALE, MlabPaja_v3:HEADER_1PIN_MALE
- removed U$2: LIPO_BATTERY400MAH, MlabPaja_v3:LIPO_BATTERY400MAH
Connections:
- removed net INT0: INT_INT1X_ACCEL.1, U2.PB5(SCK)-D13
- removed net INT1: INT_DRDYG_GYRO.1, U2.PD4(XCK/T0)-D4
- net INT2: no longer INT_INT2X_MAG.1
Changed lines of the file:
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@@
 <part name="D4" library="SparkFun-LED" deviceset="LED" device="1206" value="Green"/>
 <part name="D5" library="SparkFun-LED" deviceset="LED" device="1206" value="Orange"/>
-<part name="U$2" library="MlabPaja_v3" deviceset="LIPO_BATTERY" device="400MAH" value="LIPO_BATTERY400MAH"/>
 <part name="U$5" library="MlabPaja_v3" deviceset="VIBRATION_MOTOR" device="" value="VIBRATION_MOTOR"/>
 <part name="GND8" library="SparkFun-Aesthetics" deviceset="GND" device=""/>
@@
 <part name="BAT+2" library="MlabPaja_v3" deviceset="LIPO_PAD" device=""/>
 <part name="BAT-1" library="MlabPaja_v3" deviceset="LIPO_PAD" device=""/>
-<part name="INT_INT1X_ACCEL" library="MlabPaja_v3" deviceset="HEADER_1PIN_MALE" device=""/>
 <part name="GND_SIDE" library="MlabPaja_v3" deviceset="HEADER_1PIN_MALE" device=""/>
 <part name="SDA_SIDE" library="MlabPaja_v3" deviceset="HEADER_1PIN_MALE" device=""/>
 <part name="SCL_SIDE" library="MlabPaja_v3" deviceset="HEADER_1PIN_MALE" device=""/>
 <part name="3V3_SIDE" library="MlabPaja_v3" deviceset="HEADER_1PIN_MALE" device=""/>
-<part name="INT_DRDYG_GYRO" library="MlabPaja_v3" deviceset="HEADER_1PIN_MALE" device=""/>
 <part name="GND3" library="SparkFun-Aesthetics" deviceset="GND" device=""/>
 <part name="SUPPLY8" library="SparkFun-Aesthetics" deviceset="3.3V" device=""/>
@@
 <part name="GND6" library="SparkFun-Aesthetics" deviceset="GND" device=""/>
 <part name="GND11" library="SparkFun-Aesthetics" deviceset="GND" device=""/>
-<part name="INT_INT2X_MAG" library="MlabPaja_v3" deviceset="HEADER_1PIN_MALE" device=""/>
 </parts>
 <sheets>
@@
 <instance part="D4" gate="G$1" x="101.6" y="154.94"/>
 <instance part="D5" gate="G$1" x="111.76" y="147.32"/>
-<instance part="U$2" gate="G$1" x="101.6" y="218.44"/>
 <instance part="U$5" gate="G$1" x="248.92" y="104.14"/>
 <instance part="GND8" gate="1" x="264.16" y="93.98"/>
@@
 <instance part="BAT+2" gate="G$1" x="81.28" y="233.68" rot="R90"/>
 <instance part="BAT-1" gate="G$1" x="88.9" y="233.68" rot="R90"/>
-<instance part="INT_INT1X_ACCEL" gate="G$1" x="355.6" y="35.56"/>
 <instance part="GND_SIDE" gate="G$1" x="355.6" y="60.96"/>
 <instance part="SDA_SIDE" gate="G$1" x="355.6" y="50.8"/>
 <instance part="SCL_SIDE" gate="G$1" x="355.6" y="55.88"/>
 <instance part="3V3_SIDE" gate="G$1" x="355.6" y="45.72"/>
-<instance part="INT_DRDYG_GYRO" gate="G$1" x="355.6" y="40.64"/>
 <instance part="GND3" gate="1" x="325.12" y="33.02"/>
 <instance part="SUPPLY8" gate="G$1" x="172.72" y="137.16"/>
@@
 <instance part="GND6" gate="1" x="243.84" y="15.24"/>
 <instance part="GND11" gate="1" x="236.22" y="15.24"/>
-<instance part="INT_INT2X_MAG" gate="G$1" x="355.6" y="30.48"/>
 </instances>
 <busses>
@@
 </segment>
 </net>
-<net name="INT1" class="0">
-<segment>
-<pinref part="INT_DRDYG_GYRO" gate="G$1" pin="1"/>
-<wire x1="353.06" y1="40.64" x2="337.82" y2="40.64" width="0.1524" layer="91"/>
-<label x="337.82" y="40.64" size="1.778" layer="95"/>
-</segment>
-<segment>
-<pinref part="U2" gate="G$1" pin="PD4(XCK/T0)-D4"/>
-<wire x1="101.6" y1="53.34" x2="127" y2="53.34" width="0.1524" layer="91"/>
-<label x="121.92" y="53.34" size="1.778" layer="95"/>
-</segment>
-</net>
 <net name="VCC" class="0">
 <segment>
@@
 </segment>
 </net>
-<net name="INT0" class="0">
-<segment>
-<pinref part="U2" gate="G$1" pin="PB5(SCK)-D13"/>
-<wire x1="101.6" y1="27.94" x2="127" y2="27.94" width="0.1524" layer="91"/>
-<label x="121.92" y="27.94" size="1.778" layer="95"/>
-</segment>
-<segment>
-<pinref part="INT_INT1X_ACCEL" gate="G$1" pin="1"/>
-<wire x1="353.06" y1="35.56" x2="337.82" y2="35.56" width="0.1524" layer="91"/>
-<label x="337.82" y="35.56" size="1.778" layer="95"/>
-</segment>
-</net>
 <net name="N$1" class="0">
 <segment>
@@
 <label x="121.92" y="68.58" size="1.778" layer="95"/>
 </segment>
-<segment>
-<pinref part="INT_INT2X_MAG" gate="G$1" pin="1"/>
-<wire x1="353.06" y1="30.48" x2="337.82" y2="30.48" width="0.1524" layer="91"/>
-<label x="337.82" y="30.48" size="1.778" layer="95"/>
-</segment>
-</net>
+</net>
