File: eagle/custom_pcb/IoT_modules_atmega328_kinemata_v2.sch (EAGLE design)
At the start: 54 parts, among them IC2 4093DT, Q3 MOSFET-P, T1 2N2222, U2 ATMEGA328P, U3 FT232RL-BASICSSOP, U4 MCP73831, Y2 8MHz

Commit message: custom PCB wiring technically done, DRC ok
Connections:
- removed net INT2: U2.ADC7
- removed net RGB_B: U2.PD3(INT1)-D3~
- net LED_B: now also U2.PD3(INT1)-D3~
Changed lines of the file:
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@@
-</segment>
-</net>
-<net name="RGB_B" class="0">
-<segment>
-<pinref part="U2" gate="G$1" pin="PD3(INT1)-D3~"/>
-<wire x1="101.6" y1="55.88" x2="127" y2="55.88" width="0.1524" layer="91"/>
-<label x="121.92" y="55.88" size="1.778" layer="95"/>
 </segment>
 </net>
@@
 <label x="251.46" y="60.96" size="1.778" layer="95"/>
 </segment>
-</net>
-<net name="INT2" class="0">
-<segment>
-<pinref part="U2" gate="G$1" pin="ADC7"/>
-<wire x1="101.6" y1="68.58" x2="127" y2="68.58" width="0.1524" layer="91"/>
-<label x="121.92" y="68.58" size="1.778" layer="95"/>
-</segment>
-</net>
+<segment>
+<pinref part="U2" gate="G$1" pin="PD3(INT1)-D3~"/>
+<wire x1="101.6" y1="55.88" x2="127" y2="55.88" width="0.1524" layer="91"/>
+<label x="121.92" y="55.88" size="1.778" layer="95"/>
+</segment>
+</net>
