File: eagle/custom_pcb/IoT_modules_atmega328_kinemata_v3.sch (EAGLE design)
At the start: 54 parts, among them IC2 4093DT, Q3 MOSFET-P, T1 2N2222, U2 ATMEGA328P, U3 FT232RL-BASICSSOP, U4 MCP73831, Y2 8MHz

Commit message: custom pcb wiring passing drc
Parts:
- removed U$6: LIPO_BATTERY300MAH, MlabPaja_v3:LIPO_BATTERY300MAH
- removed U$7: LIPO_BATTERY400MAH, MlabPaja_v3:LIPO_BATTERY400MAH
- removed U$8: LIPO_BATTERY600MAH, MlabPaja_v3:LIPO_BATTERY600MAH
- removed U$9: LIPO_BATTERY900MAH, MlabPaja_v3:LIPO_BATTERY900MAH
Changed lines of the file:
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@@
 <part name="JP1" library="SparkFun-Connectors" deviceset="M04" device="LONGPADS"/>
 <part name="U$2" library="MlabPaja_v3" deviceset="LIPO_BATTERY" device="110MAH"/>
-<part name="U$6" library="MlabPaja_v3" deviceset="LIPO_BATTERY" device="300MAH"/>
-<part name="U$7" library="MlabPaja_v3" deviceset="LIPO_BATTERY" device="400MAH"/>
-<part name="U$8" library="MlabPaja_v3" deviceset="LIPO_BATTERY" device="600MAH"/>
-<part name="U$9" library="MlabPaja_v3" deviceset="LIPO_BATTERY" device="900MAH"/>
 </parts>
 <sheets>
@@
 <instance part="JP1" gate="G$1" x="355.6" y="55.88" rot="R180"/>
 <instance part="U$2" gate="G$1" x="292.1" y="99.06"/>
-<instance part="U$6" gate="G$1" x="309.88" y="99.06"/>
-<instance part="U$7" gate="G$1" x="332.74" y="91.44"/>
-<instance part="U$8" gate="G$1" x="350.52" y="93.98"/>
-<instance part="U$9" gate="G$1" x="307.34" y="83.82"/>
 </instances>
 <busses>
