File: eagle/custom_pcb/kinemata.brd (EAGLE design)
At the start: 50 x 35 mm, 54 parts, among them IC2 4093DT, Q3 MOSFET-P, T1 2N2222, U2 ATMEGA328P, U3 FT232RL-BASICSSOP, U4 MCP73831, Y2 8MHz

Commit message: added eagle design files for v4 prototype PCB
Parts:
- removed U$6: LIPO_BATTERY300MAH, MlabPaja_v3:LIPO_BATTERY_300MAH_FARNELL_2077884
- removed U$7: LIPO_BATTERY400MAH, MlabPaja_v3:LIPO_BATTERY_400MAH
- removed U$8: LIPO_BATTERY600MAH, MlabPaja_v3:LIPO_BATTERY_600MAH_FARNELL_2077883
- removed U$9: LIPO_BATTERY900MAH, MlabPaja_v3:LIPO_BATTERY_900MAH
- moved R13 17.1 mm to (41.4, 20.3), flipped to the top, turned to 180 degrees
- moved R8 12.6 mm to (41.4, 18.3), flipped to the top, turned to 180 degrees
- moved D5 10.3 mm to (48.5, 21.0)
- moved R12 9.85 mm to (32.2, 30.0), turned to 0 degrees
- moved R3 8.53 mm to (41.4, 16.3), flipped to the top, turned to 180 degrees
- moved U$5 6.87 mm to (15.1, 26.1), turned to 0 degrees
- moved BAT-1 5.86 mm to (49.5, 24.9)
- moved JP1 5.75 mm to (48.0, 16.5), flipped to the bottom, turned to 270 degrees
- moved IC2 5.62 mm to (42.9, 31.4), turned to 90 degrees
- moved D11 5.14 mm to (46.1, 21.0), turned to 90 degrees
- moved C12 4.76 mm to (36.6, 24.5), turned to 0 degrees
- moved R22 3.74 mm to (49.6, 30.5), turned to 90 degrees
- moved C8 3.51 mm to (23.3, 31.7), turned to 180 degrees
- moved R21 3.31 mm to (34.0, 27.7), flipped to the bottom
- moved R6 2.72 mm to (24.3, 16.9), flipped to the bottom, turned to 90 degrees
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Routing:
- net 3.3V: track 114.7 -> 92.2 mm, vias 6 -> 5
- net N$13: track 68.5 -> 55.5 mm, vias 2 -> 4
- net SDA: track 59.8 -> 47.1 mm
- net GND: track 216.5 -> 206.0 mm, vias 5 -> 16
- net SCL: track 44.6 -> 35.1 mm, vias 2 -> 1
- net STAT: track 28.0 -> 19.4 mm, vias 1 -> 2
- net PWR2: track 17.7 -> 26.2 mm, vias 0 -> 2
- net 5V: track 102.1 -> 93.9 mm, vias 5 -> 4
- net N$17: track 71.8 -> 64.2 mm, vias 2 -> 5
- net VIBE: track 28.2 -> 20.8 mm, vias 2 -> 1
- net VCC: track 42.6 -> 49.3 mm, vias 7 -> 5
- net N$18: track 28.2 -> 22.2 mm, vias 1 -> 2
- net N$4: track 4.84 -> 10.8 mm, vias 0 -> 1
- net N$7: track 8.40 -> 14.1 mm, vias 1 -> 2
- net LED_R: track 9.45 -> 15.0 mm, vias 0 -> 2
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Other:
- board size 50 x 35 mm -> 51 x 35 mm
