File: eagle/custom_pcb/kinemata.sch (EAGLE design)
At the start: 55 parts, among them IC2 4093DT, Q3 MOSFET-P, T1 2N2222, U1 SFW6R-3STE1LF, U2 ATMEGA328P, U3 FT232RL-BASICSSOP, U4 MCP73831, Y2 8MHz

Commit message: added eagle design files for v4 prototype PCB
Parts:
- removed 3V3_SIDE, GND_SIDE, SCL_SIDE, SDA_SIDE: HEADER_1PIN_MALE, MlabPaja_v3:HEADER_1PIN_MALE
- removed BAT+1, BAT-2: LIPO_PAD, MlabPaja_v3:LIPO_PAD
- removed U1: SFW6R-3STE1LF, MlabPaja_v3:SFW6R-3STE1LF
- added JP1: (no value), SparkFun-Connectors:M04LONGPADS
- added U$2: LIPO_BATTERY110MAH, MlabPaja_v3:LIPO_BATTERY110MAH
Connections:
- removed net INT2: U2.ADC7
- removed net RGB_B: U2.PD3(INT1)-D3~
- net 3.3V: now also JP1.2; no longer 3V3_SIDE.1
- net 5V: no longer U1.1
- net D+USB: no longer U1.3
- net D-USB: no longer U1.2
- net GND: now also JP1.1; no longer BAT-2.P$1, GND_SIDE.1, U1.4
- net LED_B: now also U2.PD3(INT1)-D3~
- net PWR1: no longer U1.5
- net PWR2: no longer U1.6
- net SCL: now also JP1.4; no longer SCL_SIDE.1
- net SDA: now also JP1.3; no longer SDA_SIDE.1
- net VCC: no longer BAT+1.P$1
